Commit message: added new urdf for testing

File: tests/urdf/awesome_leg_floating.urdf (robot description, URDF)
Before this commit: robot awesome_leg, 3 links, 2 joints
Links:
- added link base_link, mass 6.5477704; collision mesh filename=package://awesome_leg/description/new_meshes/collision/base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 scale=0.1 0.1 0.1; visual mesh filename=package://awesome_leg/description/new_meshes/visual/base.stl scale=0.1 0.1 0.1
- added link world
Joints:
- added joint hip_pitch_1: type revolute, parent base_link, child femur1, origin xyz=0 0.21459999999999999 0, axis 0 1 0, limit lower=-2.4 upper=2.4 effort=112 velocity=20.0
- added joint world_test_rig: type floating, parent world, child base_link, origin xyz=0.18 0 0.75 rpy=0.0 0.0 -1.57079632679
